File: Platinenentwurf/testboard/protoBoardHB.brd (EAGLE design)
At the start: 85 x 49.9 mm, 38 parts, among them IC1 CD74HCT125M, J1 M20-9980545, U2 STM32F4X5RG

Commit message: Platinenzeugs + Boardbilder zur ueberpruefung
Parts:
- added Q1: SMMBT3904WT1G, SamacSys_Parts:SOT65P220X100-3N
- added R1, R2, R3, R4, R5, R6, R7, R8: (no value), adafruit:R1206
- added R_SMM_1, R_SMM_2: 100K, adafruit:R1206
- moved CAN_T 17.2 mm to (70.4, 48.9)
- moved C_HB_VS_1 17.2 mm to (27.3, 35.6)
- moved C_HB_VS_2 17.2 mm to (10.8, 35.6)
- moved C_Q_1 17.2 mm to (46.2, 41.0)
- moved C_VCAP_1 17.2 mm to (60.8, 36.6)
- moved C_VDD_1 17.2 mm to (53.2, 56.9)
- moved C_VDD_2 17.2 mm to (55.8, 36.6)
- moved C_VDD_3 17.2 mm to (64.7, 36.6)
- moved C_VDD_47 17.2 mm to (49.1, 53.1)
- moved C_VR33_VIN 17.2 mm to (61.2, 27.7)
- moved C_VR33_VO1 17.2 mm to (51.0, 27.7)
- moved C_VR5_VIN 17.2 mm to (75.1, 27.7)
- moved C_VR5_VO1 17.2 mm to (65.0, 27.7)
- moved R_CD 17.2 mm to (32.4, 23.5)
- moved R_HB_INH_1 17.2 mm to (5.71, 35.6)
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Connections:
- new net OUT_PA4: R3.1
- new net OUT_PA5: R5.1
- new net OUT_PB1: R7.1
- new net PA0: R1.1, R2.2, U2.14
- new net PA4: R3.2, R4.1, U2.20
- new net PA5: R5.2, R6.1, U2.21
- new net PA8: Q1.3, R_SMM_1.2, U2.41
- new net PB1: R7.2, R8.1, U2.27
- new net SS_VN: Q1.1, R_SMM_2.1
- new net SS_VP: R_SMM_1.1
- net GND: now also Q1.2, R1.2, R4.2, R6.2, R8.2, R_SMM_2.2
- net IS_1: now also HB_ST.3, U2.8; no longer HB_ST.1, U2.17
- net IS_2: now also HB_ST.1, U2.9; no longer HB_ST.3, U2.20
- net V12: now also R2.1
Routing:
- net IS_2: track 58.7 -> 62.3 mm, vias 3 -> 2
- net IS_1: track 78.2 -> 81.7 mm, vias 4 -> 3
Other:
- board size 85 x 49.9 mm -> 109.8 x 67.7 mm
