File: Platinenentwurf/testboard/protoBoardHB.sch (EAGLE design)
At the start: 24 parts, among them U2 STM32F4X5RG

Commit message: ProtoBoard update
Parts:
- added C_HB_VS_1, C_HB_VS_2: 0.47uF, adafruit:C-USC1206
- added HB_1, HB_2: BTN8982TA, SamacSys_Parts:BTN8982TA
- added MOTOR: 282836-2, SamacSys_Parts:282836-2
- added R_HB_INH_1, R_HB_INH_2, R_HB_IN_1, R_HB_IN_2: 10K, adafruit:R-US_R1206
- added R_HB_IS_1, R_HB_IS_2: 1k, adafruit:R-US_R1206
Connections:
- removed net N$11: HB_ST.8
- new net N$3: HB_1.IN, R_HB_IN_1.2
- new net N$4: HB_1.INH, R_HB_INH_1.2
- new net N$5: HB_2.IN, R_HB_IN_2.2
- new net N$6: HB_2.INH, R_HB_INH_2.2
- new net V_MOT_MIN: HB_2.OUT_TAB, MOTOR.2
- new net V_MOT_PL: HB_1.OUT_TAB, MOTOR.1
- net GND: now also C_HB_VS_1.2, C_HB_VS_2.2, HB_1.GND, HB_1.SR, HB_2.GND, HB_2.SR, HB_ST.8, R_HB_IS_1.1, R_HB_IS_2.1; no longer HB_ST.10
- net INH: now also HB_ST.10, R_HB_INH_1.1, R_HB_INH_2.1
- net IN_1: now also R_HB_IN_1.1
- net IN_2: now also R_HB_IN_2.1
- net IS_1: now also HB_1.IS, R_HB_IS_1.2
- net IS_2: now also HB_2.IS, R_HB_IS_2.2
- net V12: now also C_HB_VS_1.1, C_HB_VS_2.1, HB_1.VS, HB_2.VS
