File: Platinenentwurf/testboard/protoBoardHB.sch (EAGLE design)
At the start: 38 parts, among them IC1 CD74HCT125M, J1 M20-9980545, U2 STM32F4X5RG

Commit message: Platinenzeugs + Boardbilder zur ueberpruefung
Parts:
- added Q1: SMMBT3904WT1G, SamacSys_Parts:SMMBT3904WT1G
- added R1, R2, R3, R4, R5, R6, R7, R8: (no value), adafruit:R-US_R1206
- added R_SMM_1, R_SMM_2: 100K, adafruit:R-US_R1206
Connections:
- new net OUT_PA4: R3.1
- new net OUT_PA5: R5.1
- new net OUT_PB1: R7.1
- new net PA0: R1.1, R2.2, U2A.PA0/WKUP
- new net PA4: R3.2, R4.1, U2A.PA4
- new net PA5: R5.2, R6.1, U2A.PA5
- new net PA8: Q1.C, R_SMM_1.2, U2A.PA8
- new net PB1: R7.2, R8.1, U2A.PB1
- new net SS_VN: Q1.B, R_SMM_2.1
- new net SS_VP: R_SMM_1.1
- net GND: now also Q1.E, R1.2, R4.2, R6.2, R8.2, R_SMM_2.2
- net IS_1: now also HB_ST.3, U2A.PC0; no longer HB_ST.1, U2A.PA3
- net IS_2: now also HB_ST.1, U2A.PC1; no longer HB_ST.3, U2A.PA4
- net V12: now also R2.1
