File: Platinenentwurf/testboard/protoBoardLogic.brd (EAGLE design)
At the start: 50 x 46.9 mm, 24 parts, among them U2 STM32F4X5RG

Commit message: ProtoBoard update
Connections:
- removed net N$11: HB_ST.8
- net GND: now also HB_ST.8; no longer HB_ST.10
- net INH: now also HB_ST.10
Routing:
- net GND: track 196.1 -> 190.8 mm
Changed lines of the file:
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@@
 <contactref element="SWD" pad="7"/>
 <contactref element="SWD" pad="9"/>
-<contactref element="HB_ST" pad="10"/>
 <wire x1="33.02" y1="36.96" x2="35.56" y2="36.96" width="0.2032" layer="1"/>
 <wire x1="30.48" y1="36.96" x2="33.02" y2="36.96" width="0.2032" layer="1"/>
@@
 <wire x1="13.25" y1="18.92" x2="14.605" y2="18.92" width="0.254" layer="1"/>
 <wire x1="12.065" y1="20.105" x2="9.8425" y2="17.8825" width="0.254" layer="1"/>
-<wire x1="9.8425" y1="17.8825" x2="9.8425" y2="16.1925" width="0.254" layer="1"/>
 <wire x1="16.8275" y1="6.22" x2="14.4175" y2="3.81" width="0.254" layer="1"/>
 <wire x1="8.255" y1="3.81" x2="7.3025" y2="4.7625" width="0.254" layer="1"/>
 <wire x1="7.3025" y1="4.7625" x2="7.3025" y2="13.6525" width="0.254" layer="1"/>
-<wire x1="7.3025" y1="13.6525" x2="9.8425" y2="16.1925" width="0.254" layer="1"/>
 <wire x1="14.4175" y1="3.81" x2="8.255" y2="3.81" width="0.254" layer="1"/>
 <wire x1="29.21" y1="44.45" x2="30.48" y2="43.18" width="0.254" layer="1"/>
@@
 <vertex x="0.3175" y="47.9425"/>
 </polygon>
+<contactref element="HB_ST" pad="8"/>
+<wire x1="9.8425" y1="13.6525" x2="9.8425" y2="17.8825" width="0" layer="19" extent="1-1"/>
+<wire x1="7.3025" y1="13.6525" x2="9.8425" y2="13.6525" width="0" layer="19" extent="1-1"/>
 </signal>
 <signal name="CAN1_RX">
@@
 <wire x1="18.38" y1="25.92" x2="16.7125" y2="25.92" width="0.2" layer="1"/>
 <wire x1="16.7125" y1="25.92" x2="16.1925" y2="25.4" width="0.2" layer="1"/>
+<contactref element="HB_ST" pad="10"/>
+<wire x1="9.8425" y1="16.1925" x2="12.3825" y2="16.1925" width="0" layer="19" extent="1-1"/>
 </signal>
 <signal name="IN_1">
@@
 <wire x1="21.88" y1="22.2525" x2="21.2725" y2="22.86" width="0.2" layer="1"/>
 </signal>
-<signal name="N$11">
-<contactref element="HB_ST" pad="8"/>
-</signal>
 <signal name="V12">
