File: Platinenentwurf/testboard/protoBoardLogic.sch (EAGLE design)
At the start: 24 parts, among them U2 STM32F4X5RG

Commit message: ProtoBoard update
Connections:
- removed net N$11: HB_ST.8
- net GND: now also HB_ST.8; no longer HB_ST.10
- net INH: now also HB_ST.10
Changed lines of the file:
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@@
 </instance>
 <instance part="HB_ST" gate="G$1" x="-33.02" y="73.66" smashed="yes" rot="MR0">
-<attribute name="NAME" x="-31.75" y="83.82" size="1.778" layer="95" rot="MR0" align="center-left"/>
 <attribute name="VALUE" x="-31.75" y="81.28" size="1.778" layer="96" rot="MR0" align="center-left"/>
 <attribute name="OC_FARNELL" x="-33.02" y="73.66" size="1.778" layer="96" rot="MR0" display="off"/>
@@
 </segment>
 <segment>
-<pinref part="HB_ST" gate="G$1" pin="10"/>
-<wire x1="-55.88" y1="63.5" x2="-58.42" y2="63.5" width="0.1524" layer="91"/>
-<wire x1="-58.42" y1="63.5" x2="-58.42" y2="58.42" width="0.1524" layer="91"/>
-<wire x1="-58.42" y1="58.42" x2="-63.5" y2="58.42" width="0.1524" layer="91"/>
-<label x="-63.5" y="58.42" size="1.778" layer="95" rot="R180" xref="yes"/>
+<pinref part="HB_ST" gate="G$1" pin="8"/>
+<wire x1="-55.88" y1="66.04" x2="-60.96" y2="66.04" width="0.1524" layer="91"/>
+<wire x1="-60.96" y1="66.04" x2="-60.96" y2="63.5" width="0.1524" layer="91"/>
+<wire x1="-60.96" y1="63.5" x2="-63.5" y2="63.5" width="0.1524" layer="91"/>
+<label x="-63.5" y="63.5" size="1.778" layer="95" rot="R180" xref="yes"/>
 </segment>
 </net>
@@
 <label x="-25.4" y="58.42" size="1.778" layer="95" xref="yes"/>
 </segment>
+<segment>
+<pinref part="HB_ST" gate="G$1" pin="10"/>
+<wire x1="-55.88" y1="63.5" x2="-58.42" y2="63.5" width="0.1524" layer="91"/>
+<wire x1="-58.42" y1="63.5" x2="-58.42" y2="58.42" width="0.1524" layer="91"/>
+<wire x1="-58.42" y1="58.42" x2="-63.5" y2="58.42" width="0.1524" layer="91"/>
+<label x="-63.5" y="58.42" size="1.778" layer="95" rot="R180" xref="yes"/>
+</segment>
 </net>
 <net name="IN_1" class="0">
@@
 </segment>
 </net>
-<net name="N$11" class="0">
-<segment>
-<pinref part="HB_ST" gate="G$1" pin="8"/>
-<wire x1="-55.88" y1="66.04" x2="-60.96" y2="66.04" width="0.1524" layer="91"/>
-<wire x1="-60.96" y1="66.04" x2="-60.96" y2="63.5" width="0.1524" layer="91"/>
-<wire x1="-60.96" y1="63.5" x2="-63.5" y2="63.5" width="0.1524" layer="91"/>
-<label x="-63.5" y="63.5" size="1.778" layer="95" rot="R180" xref="yes"/>
-</segment>
-</net>
