File: Platinenentwurf/testboard/ProtoBoardHB/protoBoardHB.sch (EAGLE design)
At the start: 49 parts, among them IC1 CD74HCT125M, J1 M20-9980545, Q1 SMMBT3904WT1G, U2 STM32F4X5RG

Commit message: Platinenentwurf: kleines Update
Parts:
- added J2: M20-9980545, SamacSys_Parts:M20-9980545
Connections:
- removed net SS_VP: R_SMM_1.1
- new net N$15: J2.6
- new net N$16: J2.8
- new net N$17: J2.10
- new net OUT_PA6: J2.5
- net GND: now also J2.4
- net IS_1: now also HB_ST.3; no longer HB_ST.1
- net IS_2: now also HB_ST.1; no longer HB_ST.3
- net OUT_PA4: now also J2.7
- net OUT_PA5: now also J2.3
- net OUT_PB1: now also J2.1
- net PA0: now also U2A.PA0/WKUP
- net SS_VN: now also J2.2
- net V33: now also J2.9, R_SMM_1.1
Changed lines of the file:
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@@
 </variantdefs>
 <classes>
-<class number="0" name="default" width="0.2" drill="0.5">
+<class number="0" name="default" width="0.2" drill="0.508">
+</class>
+<class number="1" name="V12" width="0.6" drill="0.8">
 </class>
 </classes>
@@
 <part name="R8" library="adafruit" library_urn="urn:adsk.eagle:library:420" deviceset="R-US_" device="R1206" package3d_urn="urn:adsk.eagle:package:6240569/1"/>
 <part name="GND18" library="supply1" library_urn="urn:adsk.eagle:library:371" deviceset="GND" device=""/>
+<part name="J2" library="SamacSys_Parts" deviceset="M20-9980545" device=""/>
 </parts>
 <sheets>
@@
 <instance part="GND18" gate="1" x="279.4" y="180.34" smashed="yes">
 <attribute name="VALUE" x="279.4" y="177.8" size="1.778" layer="96"/>
+</instance>
+<instance part="J2" gate="G$1" x="220.98" y="266.7" smashed="yes">
+<attribute name="NAME" x="227.33" y="274.32" size="1.778" layer="95" align="center-left"/>
+<attribute name="VALUE" x="227.33" y="271.78" size="1.778" layer="96" align="center-left"/>
 </instance>
 </instances>
@@
 <wire x1="279.4" y1="190.5" x2="279.4" y2="182.88" width="0.1524" layer="91"/>
 </segment>
+<segment>
+<pinref part="J2" gate="G$1" pin="4"/>
+<wire x1="243.84" y1="264.16" x2="248.92" y2="264.16" width="0.1524" layer="91"/>
+<wire x1="248.92" y1="264.16" x2="248.92" y2="266.7" width="0.1524" layer="91"/>
+<wire x1="248.92" y1="266.7" x2="251.46" y2="266.7" width="0.1524" layer="91"/>
+<label x="251.46" y="266.7" size="1.778" layer="95" xref="yes"/>
+</segment>
 </net>
 <net name="CAN1_RX" class="0">
@@
 </net>
 <net name="IS_1" class="0">
-<segment>
-<pinref part="HB_ST" gate="G$1" pin="1"/>
-<wire x1="-33.02" y1="73.66" x2="-30.48" y2="73.66" width="0.1524" layer="91"/>
-<wire x1="-30.48" y1="73.66" x2="-30.48" y2="78.74" width="0.1524" layer="91"/>
-<wire x1="-30.48" y1="78.74" x2="-25.4" y2="78.74" width="0.1524" layer="91"/>
-<label x="-25.4" y="78.74" size="1.778" layer="95" xref="yes"/>
-</segment>
 <segment>
 <pinref part="R_HB_IS_1" gate="G$1" pin="2"/>
@@
 <label x="121.92" y="76.2" size="1.778" layer="95" xref="yes"/>
 </segment>
-</net>
-<net name="IS_2" class="0">
 <segment>
 <pinref part="HB_ST" gate="G$1" pin="3"/>
@@
 <label x="-25.4" y="73.66" size="1.778" layer="95" xref="yes"/>
 </segment>
+</net>
+<net name="IS_2" class="0">
 <segment>
 <pinref part="HB_2" gate="G$1" pin="IS"/>
@@
 <wire x1="116.84" y1="71.12" x2="121.92" y2="71.12" width="0.1524" layer="91"/>
 <label x="121.92" y="71.12" size="1.778" layer="95" xref="yes"/>
+</segment>
+<segment>
+<pinref part="HB_ST" gate="G$1" pin="1"/>
+<wire x1="-33.02" y1="73.66" x2="-30.48" y2="73.66" width="0.1524" layer="91"/>
+<wire x1="-30.48" y1="73.66" x2="-30.48" y2="78.74" width="0.1524" layer="91"/>
+<wire x1="-30.48" y1="78.74" x2="-25.4" y2="78.74" width="0.1524" layer="91"/>
+<label x="-25.4" y="78.74" size="1.778" layer="95" xref="yes"/>
 </segment>
 </net>
@@
 <label x="-63.5" y="68.58" size="1.778" layer="95" rot="R180" xref="yes"/>
 </segment>
+<segment>
+<pinref part="R_SMM_1" gate="G$1" pin="1"/>
+<wire x1="111.76" y1="233.68" x2="111.76" y2="236.22" width="0.1524" layer="91"/>
+<label x="111.76" y="241.3" size="1.778" layer="95" rot="R90" xref="yes"/>
+<wire x1="111.76" y1="236.22" x2="111.76" y2="241.3" width="0.1524" layer="91"/>
+<wire x1="111.76" y1="236.22" x2="88.9" y2="236.22" width="0.1524" layer="91"/>
+<junction x="111.76" y="236.22"/>
+<label x="88.9" y="236.22" size="1.778" layer="95" rot="R180" xref="yes"/>
+</segment>
+<segment>
+<pinref part="J2" gate="G$1" pin="9"/>
+<wire x1="220.98" y1="256.54" x2="218.44" y2="256.54" width="0.1524" layer="91"/>
+<wire x1="218.44" y1="256.54" x2="218.44" y2="251.46" width="0.1524" layer="91"/>
+<wire x1="218.44" y1="251.46" x2="213.36" y2="251.46" width="0.1524" layer="91"/>
+<label x="213.36" y="251.46" size="1.778" layer="95" rot="R180" xref="yes"/>
+</segment>
 </net>
 <net name="V5" class="0">
@@
 <label x="88.9" y="210.82" size="1.778" layer="95" rot="R180" xref="yes"/>
 </segment>
-</net>
-<net name="SS_VP" class="0">
-<segment>
-<pinref part="R_SMM_1" gate="G$1" pin="1"/>
-<wire x1="111.76" y1="233.68" x2="111.76" y2="236.22" width="0.1524" layer="91"/>
-<label x="111.76" y="241.3" size="1.778" layer="95" rot="R90" xref="yes"/>
-<wire x1="111.76" y1="236.22" x2="111.76" y2="241.3" width="0.1524" layer="91"/>
-<wire x1="111.76" y1="236.22" x2="88.9" y2="236.22" width="0.1524" layer="91"/>
-<junction x="111.76" y="236.22"/>
-<label x="88.9" y="236.22" size="1.778" layer="95" rot="R180" xref="yes"/>
+<segment>
+<pinref part="J2" gate="G$1" pin="2"/>
+<wire x1="243.84" y1="266.7" x2="246.38" y2="266.7" width="0.1524" layer="91"/>
+<wire x1="246.38" y1="266.7" x2="246.38" y2="271.78" width="0.1524" layer="91"/>
+<wire x1="246.38" y1="271.78" x2="251.46" y2="271.78" width="0.1524" layer="91"/>
+<label x="251.46" y="271.78" size="1.778" layer="95" xref="yes"/>
 </segment>
 </net>
@@
 <label x="208.28" y="203.2" size="1.778" layer="95" xref="yes"/>
 </segment>
+<segment>
+<pinref part="U2" gate="A" pin="PA0/WKUP"/>
+<wire x1="50.8" y1="66.04" x2="48.26" y2="66.04" width="0.1524" layer="91"/>
+<wire x1="48.26" y1="66.04" x2="48.26" y2="73.66" width="0.1524" layer="91"/>
+<wire x1="48.26" y1="73.66" x2="40.64" y2="73.66" width="0.1524" layer="91"/>
+<label x="40.64" y="73.66" size="1.778" layer="95" rot="R180" xref="yes"/>
+</segment>
 </net>
 <net name="PA4" class="0">
@@
 <label x="231.14" y="220.98" size="1.778" layer="95" rot="R90" xref="yes"/>
 </segment>
+<segment>
+<pinref part="J2" gate="G$1" pin="7"/>
+<wire x1="220.98" y1="259.08" x2="215.9" y2="259.08" width="0.1524" layer="91"/>
+<wire x1="215.9" y1="259.08" x2="215.9" y2="256.54" width="0.1524" layer="91"/>
+<wire x1="215.9" y1="256.54" x2="213.36" y2="256.54" width="0.1524" layer="91"/>
+<label x="213.36" y="256.54" size="1.778" layer="95" rot="R180" xref="yes"/>
+</segment>
 </net>
 <net name="OUT_PA5" class="0">
@@
 <label x="259.08" y="220.98" size="1.778" layer="95" rot="R90" xref="yes"/>
 </segment>
+<segment>
+<pinref part="J2" gate="G$1" pin="3"/>
+<wire x1="220.98" y1="264.16" x2="215.9" y2="264.16" width="0.1524" layer="91"/>
+<wire x1="215.9" y1="264.16" x2="215.9" y2="266.7" width="0.1524" layer="91"/>
+<wire x1="215.9" y1="266.7" x2="213.36" y2="266.7" width="0.1524" layer="91"/>
+<label x="213.36" y="266.7" size="1.778" layer="95" rot="R180" xref="yes"/>
+</segment>
 </net>
 <net name="OUT_PB1" class="0">
@@
 <wire x1="279.4" y1="218.44" x2="279.4" y2="220.98" width="0.1524" layer="91"/>
 <label x="279.4" y="220.98" size="1.778" layer="95" rot="R90" xref="yes"/>
+</segment>
+<segment>
+<pinref part="J2" gate="G$1" pin="1"/>
+<wire x1="220.98" y1="266.7" x2="218.44" y2="266.7" width="0.1524" layer="91"/>
+<wire x1="218.44" y1="266.7" x2="218.44" y2="271.78" width="0.1524" layer="91"/>
+<wire x1="218.44" y1="271.78" x2="213.36" y2="271.78" width="0.1524" layer="91"/>
+<label x="213.36" y="271.78" size="1.778" layer="95" rot="R180" xref="yes"/>
 </segment>
 </net>
@@
 </segment>
 </net>
+<net name="OUT_PA6" class="0">
+<segment>
+<pinref part="J2" gate="G$1" pin="5"/>
+<wire x1="220.98" y1="261.62" x2="213.36" y2="261.62" width="0.1524" layer="91"/>
+<label x="213.36" y="261.62" size="1.778" layer="95" rot="R180" xref="yes"/>
+</segment>
+</net>
+<net name="N$15" class="0">
+<segment>
+<pinref part="J2" gate="G$1" pin="6"/>
+<wire x1="243.84" y1="261.62" x2="251.46" y2="261.62" width="0.1524" layer="91"/>
+</segment>
+</net>
+<net name="N$16" class="0">
+<segment>
+<pinref part="J2" gate="G$1" pin="8"/>
+<wire x1="243.84" y1="259.08" x2="248.92" y2="259.08" width="0.1524" layer="91"/>
+<wire x1="248.92" y1="259.08" x2="248.92" y2="256.54" width="0.1524" layer="91"/>
+<wire x1="248.92" y1="256.54" x2="251.46" y2="256.54" width="0.1524" layer="91"/>
+</segment>
+</net>
+<net name="N$17" class="0">
+<segment>
+<pinref part="J2" gate="G$1" pin="10"/>
+<wire x1="243.84" y1="256.54" x2="246.38" y2="256.54" width="0.1524" layer="91"/>
+<wire x1="246.38" y1="256.54" x2="246.38" y2="251.46" width="0.1524" layer="91"/>
+<wire x1="246.38" y1="251.46" x2="251.46" y2="251.46" width="0.1524" layer="91"/>
+</segment>
+</net>
