File: Platinenentwurf/testboard/ProtoBoardHB/protoBoardHB.sch (EAGLE design)
At the start: 52 parts, among them IC1 CD74HCT125M, J1 M20-9980545, J2 M20-9980545, J3 M20-9990246, J4 M20-9990246, Q1 SMMBT3904WT1G, U2 STM32F4X5RG

Commit message: update Platine
Parts:
- R17: value 100K -> 7.5K
- renumbered CAN_CONNECTION to CAN_OUT, C_HB_VS_1 to CH1, C_HB_VS_2 to CH2, C_Q_1 to CQ1, C_Q_2 to CQ2, C_VCAP_1 to C6, C_VCAP_2 to C5, C_VDDA to C12, C_VDD_1 to C10, C_VDD_2 to C7, C_VDD_3 to C8, C_VDD_4 to C9, C_VDD_47 to C11, C_VR33_VIN to C2, C_VR33_VO1 to C1, C_VR5_VIN to C4, C_VR5_VO1 to C3, IC1 to CD74HCT, J1 to J_CD, J2 to SENSORIK, J3 to J_IS2, J4 to J_IS1, QUARZ to QUARTZ, R_CD to R15, R_HB_INH_1 to R12, R_HB_INH_2 to R11, R_HB_IN_1 to R13, R_HB_IN_2 to R10, R_HB_IS_1 to R14, R_HB_IS_2 to R9, R_SMM_1 to R16, R_SMM_2 to R17, VREG_55 to VREG_5
Connections:
- removed net N$16: SENSORIK.8
- removed net N$17: SENSORIK.10

Commit message: Platinenupdate
Parts:
- added C13: 470uF, adafruit:C-US050-075X075
- added C14, C15: 1nF, adafruit:C-USC1206
- added MGT1: BEAGLEBONEBLACK_MOUNTING_HOLE, BeagleBone_Black_Wireless:BEAGLEBONEBLACK_MOUNTING_HOLE
- added R18, R19: 1k, adafruit:R-US_R1206
- renumbered CH2 to CH3
Connections:
- new net BOOT0: R19.2, U2A.BOOT0
- new net BOOT1: R18.2, U2A.PB2/BOOT1
- net GND: now also C13.2, C14.2, C15.2, MGT1.P$1, R18.1, R19.1
- net IS_1: no longer R14.2
- net IS_2: no longer R9.2
- net N$2: now also C15.1, R9.2
- net N$7: now also C14.1, R14.2
- net V12: now also C13.1
Other:
- moved on the sheet: BAT, J_IS1, J_IS2, R14, R9
