File: Platinenentwurf/testboard/Board/Board.brd (EAGLE design)
At the start: 88.8 x 50 mm, 55 parts, among them J1 1-776267-1, Q1 SMMBT3904WT1G, U2 STM32F4X5RG

Commit message: Platine
Parts:
- added IC1: 1711725, SamacSys_Parts:PHEONIX-5.08PITCH-2PIN
- moved QUARTZ 12.5 mm to (16.7, 11.1)
- moved CAN_T 11.0 mm to (16.0, 41.0)
- moved CD74HCT 6.08 mm to (29.0, 26.0)
- moved U2 4.12 mm to (15.0, 26.0)
Routing:
- added copper zone on layer 1, net V_MOT_MIN
- added copper zone on layer 1, net V_MOT_PL
