File: Platinenentwurf/testboard/Board/Board.brd (EAGLE design)
At the start: 88.8 x 50 mm, 45 parts, among them IC1 1711725, J1 1-776267-1, U2 STM32F4X5RG

Commit message: Inventarliste added
Parts:
- removed R18, R19: 1k, adafruit:R1206
- added C16, C17, C18, C19: 220nF, adafruit:C1206
- added J2, J3: 282836-2, SamacSys_Parts:SHDR2W100P0X500_1X2_1000X820X1
- added J4: M20-9990246, SamacSys_Parts:HDRV2W64P0X254_1X2_508X254X864
- added R16: 220, adafruit:R1206
- added R17: 0, adafruit:R1206
- added R5: 100, adafruit:R1206
- added R_RS: 10, adafruit:R1206
- C11: value 4.7nF -> 4.7uF
- CH1, CH3: value 0.47uF -> 100nF
- moved R10 30.0 mm to (39.0, 6.00), turned to 180 degrees
- moved R11 27.2 mm to (39.0, 9.00), turned to 180 degrees
- moved C12 7.62 mm to (32.0, 12.0), turned to 0 degrees
- moved C3 7.47 mm to (31.3, 38.6), turned to 180 degrees
- moved CQ1 6.50 mm to (26.0, 9.00), turned to 90 degrees
- moved C6 6.40 mm to (32.0, 21.0), turned to 0 degrees
- moved C4 5.66 mm to (37.0, 45.0)
- moved C2 4.47 mm to (23.0, 45.0), turned to 270 degrees
- moved C14 3.00 mm to (62.0, 46.0)
- moved CH1 3.00 mm to (59.0, 46.0)
- moved R12 3.00 mm to (56.0, 46.0)
- moved R13 3.00 mm to (53.0, 46.0)
- moved VREG_33 2.24 mm to (17.0, 44.0)
- moved CQ2 2.00 mm to (13.0, 9.00), turned to 90 degrees
- moved VREG_5 2.00 mm to (30.0, 44.0)
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Connections:
- removed net BOOT0: R19.2, U2.60
- removed net BOOT1: R18.2, U2.28
- new net CAN_RS: CAN_T.8, R_RS.1
- new net Q_IN: CQ2.1, QUARTZ.2, R17.2
- new net Q_OUT: CQ1.1, QUARTZ.1, R16.2
- net CANH: now also R5.2
- net CANL: now also R5.1
- net GND: now also C18.1, C19.1, J1.11, J3.1, R_RS.2, U2.28, U2.60; no longer CAN_T.8, R18.1, R19.1
- net INH: no longer U2.24
- net INH_M: now also U2.24
- net L_1: now also J1.13, J2.2
- net L_2: now also J1.14, J2.1
- net OSC_IN: now also R17.1; no longer CQ2.1, QUARTZ.2
- net OSC_OUT: now also R16.1; no longer CQ1.1, QUARTZ.1
- net U_RX: now also J4.1
- net U_TX: now also J4.2
- net V12: now also C16.2, C17.2
- net V33: now also J3.2; no longer CD74HCT.10
- net V5: now also J1.12
- net V_MOT_MIN: now also C17.1, C19.2
- net V_MOT_PL: now also C16.1, C18.2

Commit message: Platinenzeug
Parts:
- added C20: 1 uF, adafruit:C1206
- added R15, R18: (no value), adafruit:R1206
- moved J2 8.06 mm to (54.0, 5.00)
- moved C5 6.71 mm to (13.0, 33.0)
- moved C9 5.39 mm to (13.0, 36.0), turned to 180 degrees
- moved C_CAN 5.10 mm to (13.0, 30.0), turned to 180 degrees
- moved J3 4.12 mm to (65.0, 5.00)
- moved C18 4.00 mm to (44.0, 36.0)
- moved C1 3.00 mm to (7.00, 36.0)
- moved CQ1 3.00 mm to (23.0, 9.00)
- moved R16 3.00 mm to (20.0, 9.00)
- moved CAN_T 1.41 mm to (22.0, 34.0), turned to 0 degrees
- moved J4 1.41 mm to (38.0, 13.0), turned to 90 degrees
- moved C16 1.00 mm to (53.0, 25.0), turned to 0 degrees
- moved C19 1.00 mm to (43.0, 16.0), turned to 90 degrees
- moved U2 1.00 mm to (19.0, 20.0)
- renumbered QUARTZ to QUARZ
Connections:
- new net PC5: R15.2, R18.1, U2.25
- net GND: now also C20.2, R18.2
- net L_1: no longer J2.2
- net L_2: no longer J2.1
- net T_1: now also J2.1
- net V12: now also R15.1
- net V33: now also C20.1
- net Z_1: now also J2.2

Commit message: Platinenzeug
Parts:
- moved C4 1.41 mm to (36.0, 44.0)
- moved C2 1.00 mm to (23.0, 44.0)
Changed lines of the file:
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@@
 <attribute name="VALUE" x="70.73" y="8.587" size="1.27" layer="27"/>
 </element>
-<element name="C2" library="adafruit" library_urn="urn:adsk.eagle:library:420" package="C1206" package3d_urn="urn:adsk.eagle:package:6240335/1" value="1uF" x="23" y="45" smashed="yes" rot="R270">
-<attribute name="NAME" x="24.143" y="46.27" size="1.27" layer="25" rot="R270"/>
-<attribute name="VALUE" x="20.587" y="46.27" size="1.27" layer="27" rot="R270"/>
+<element name="C2" library="adafruit" library_urn="urn:adsk.eagle:library:420" package="C1206" package3d_urn="urn:adsk.eagle:package:6240335/1" value="1uF" x="23" y="44" smashed="yes" rot="R270">
+<attribute name="NAME" x="24.143" y="45.27" size="1.27" layer="25" rot="R270"/>
+<attribute name="VALUE" x="20.587" y="45.27" size="1.27" layer="27" rot="R270"/>
 </element>
 <element name="C3" library="adafruit" library_urn="urn:adsk.eagle:library:420" package="C1206" package3d_urn="urn:adsk.eagle:package:6240335/1" value="4.7uF" x="31.34" y="38.61" smashed="yes" rot="R180">
@@
 <attribute name="VALUE" x="32.61" y="41.023" size="1.27" layer="27" rot="R180"/>
 </element>
-<element name="C4" library="adafruit" library_urn="urn:adsk.eagle:library:420" package="C1206" package3d_urn="urn:adsk.eagle:package:6240335/1" value="1uF" x="37" y="45" smashed="yes" rot="R90">
-<attribute name="NAME" x="35.857" y="43.73" size="1.27" layer="25" rot="R90"/>
-<attribute name="VALUE" x="39.413" y="43.73" size="1.27" layer="27" rot="R90"/>
+<element name="C4" library="adafruit" library_urn="urn:adsk.eagle:library:420" package="C1206" package3d_urn="urn:adsk.eagle:package:6240335/1" value="1uF" x="36" y="44" smashed="yes" rot="R90">
+<attribute name="NAME" x="34.857" y="42.73" size="1.27" layer="25" rot="R90"/>
+<attribute name="VALUE" x="38.413" y="42.73" size="1.27" layer="27" rot="R90"/>
 </element>
 <element name="C5" library="adafruit" library_urn="urn:adsk.eagle:library:420" package="C1206" package3d_urn="urn:adsk.eagle:package:6240335/1" value="2.2uF" x="13" y="33" smashed="yes" rot="R180">
@@
 <wire x1="44" y1="37.4" x2="47.1" y2="45" width="0" layer="19" extent="1-1"/>
 <wire x1="38" y1="37.422" x2="44" y2="37.4" width="0" layer="19" extent="1-1"/>
-<wire x1="37" y1="43.6" x2="38" y2="37.422" width="0" layer="19" extent="1-1"/>
-<wire x1="32.6" y1="41.7" x2="37" y2="43.6" width="0" layer="19" extent="1-1"/>
+<wire x1="36" y1="42.6" x2="38" y2="37.422" width="0" layer="19" extent="1-1"/>
+<wire x1="32.6" y1="41.7" x2="36" y2="42.6" width="0" layer="19" extent="1-1"/>
 <wire x1="32.74" y1="38.61" x2="32.6" y2="41.7" width="0" layer="19" extent="1-1"/>
 <wire x1="33.712" y1="33.54" x2="32.74" y2="38.61" width="0" layer="19" extent="1-1"/>
@@
 <wire x1="19.5362" y1="34.635" x2="11.6" y2="36" width="0" layer="19" extent="1-1"/>
 <wire x1="19.6" y1="41.7" x2="19.5362" y2="34.635" width="0" layer="19" extent="1-1"/>
-<wire x1="23" y1="43.6" x2="19.6" y2="41.7" width="0" layer="19" extent="1-1"/>
+<wire x1="23" y1="42.6" x2="19.6" y2="41.7" width="0" layer="19" extent="1-1"/>
 <wire x1="7.1" y1="45" x2="5.6" y2="36" width="0" layer="19" extent="1-1"/>
 <wire x1="43" y1="14.6" x2="33.4" y2="15" width="0" layer="19" extent="1-1"/>
@@
 <wire x1="54.4" y1="25" x2="61.4" y2="23" width="0" layer="19" extent="1-1"/>
 <wire x1="41" y1="37.422" x2="59" y2="44.6" width="0" layer="19" extent="1-1"/>
-<wire x1="37" y1="46.4" x2="41" y2="37.422" width="0" layer="19" extent="1-1"/>
-<wire x1="32.6" y1="46.3" x2="37" y2="46.4" width="0" layer="19" extent="1-1"/>
-<wire x1="23" y1="46.4" x2="32.6" y2="46.3" width="0" layer="19" extent="1-1"/>
-<wire x1="19.6" y1="46.3" x2="23" y2="46.4" width="0" layer="19" extent="1-1"/>
+<wire x1="36" y1="45.4" x2="41" y2="37.422" width="0" layer="19" extent="1-1"/>
+<wire x1="32.6" y1="46.3" x2="36" y2="45.4" width="0" layer="19" extent="1-1"/>
+<wire x1="23" y1="45.4" x2="32.6" y2="46.3" width="0" layer="19" extent="1-1"/>
+<wire x1="19.6" y1="46.3" x2="23" y2="45.4" width="0" layer="19" extent="1-1"/>
 </signal>
 <signal name="V33">

Commit message: Platinenzeug
Parts:
- removed R16: 220, adafruit:R1206
- removed R17: 0, adafruit:R1206
- added C21: 1uF, adafruit:C1206
- added R19: 0, resistor:R0805
- added R20: 220, resistor:R0805
- added U$1: (no value), Nordic_nRF:RESC0805_N
- R14, R9: value 1k -> 0.5k
- moved R5 62.6 mm to (68.0, 47.0)
- moved C16 12.5 mm to (47.0, 36.0), turned to 90 degrees
- moved R2 7.62 mm to (39.0, 3.00)
- moved R3 7.62 mm to (32.0, 6.00)
- moved C5 7.28 mm to (6.00, 35.0)
- moved R1 6.00 mm to (32.0, 3.00), turned to 180 degrees
- moved R4 6.00 mm to (32.0, 9.00), turned to 0 degrees
- moved J4 3.00 mm to (38.0, 16.0), turned to 270 degrees
- moved R10 3.00 mm to (39.0, 9.00), turned to 0 degrees
- moved R11 3.00 mm to (39.0, 6.00), turned to 0 degrees
- moved C1 2.24 mm to (6.00, 38.0)
- moved C10 2.24 mm to (6.00, 17.0)
- moved C11 2.24 mm to (6.00, 14.0)
- moved R6 2.24 mm to (6.00, 23.0)
- moved R7 2.24 mm to (6.00, 29.0)
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Connections:
- new net VDDA: C12.1, C20.1, U$1.1, U2.13
- net CANH: now also J1.13; no longer J1.8
- net CANL: now also J1.14; no longer J1.7
- net GND: now also C21.2, J1.3, J1.8; no longer J1.11, J1.6
- net L_1: now also J1.7; no longer J1.13
- net L_2: now also J1.6; no longer J1.14
- net NRST: now also J1.11; no longer J1.10
- net OSC_IN: now also R19.2; no longer R17.1
- net OSC_OUT: now also R20.2; no longer R16.1
- net Q_IN: now also R19.1; no longer R17.2
- net Q_OUT: now also R20.1; no longer R16.2
- net SWCLK: now also J1.1; no longer J1.3
- net SWDIO: now also J1.10; no longer J1.2
- net TRACESWO: now also J1.12; no longer J1.9
- net T_1: now also C21.1
- net V33: now also J1.2, U$1.2; no longer C12.1, C20.1, J1.1, U2.13
- net V5: now also J1.9; no longer J1.12
Routing:
- net V33: track 0.00 -> 254.1 mm, vias 0 -> 2
- net IS_1: track 0.00 -> 93.9 mm, vias 0 -> 3
- net INH: track 0.00 -> 92.9 mm, vias 0 -> 3
- net TRACESWO: track 0.00 -> 90.5 mm, vias 0 -> 1
- net V12: track 0.00 -> 88.9 mm
- net Z_1: track 0.00 -> 88.4 mm, vias 0 -> 1
- net IS_2: track 0.00 -> 87.4 mm, vias 0 -> 2
- net NRST: track 0.00 -> 87.3 mm, vias 0 -> 1
- net SWDIO: track 0.00 -> 85.8 mm, vias 0 -> 1
- net V5: track 0.00 -> 82.6 mm, vias 0 -> 2
- net CANL: track 0.00 -> 81.5 mm, vias 0 -> 2
- net CANH: track 0.00 -> 80.0 mm, vias 0 -> 2
- net SWCLK: track 0.00 -> 78.9 mm, vias 0 -> 1
- net IN_1: track 0.00 -> 72.0 mm, vias 0 -> 2
- net T_1: track 0.00 -> 71.5 mm, vias 0 -> 2
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