File: Platinenentwurf/testboard/Board/Board.sch (EAGLE design)
At the start: 55 parts, among them J1 1-776267-1, Q1 SMMBT3904WT1G, U2 STM32F4X5RG

Commit message: Platine
Parts:
- added IC1: 1711725, SamacSys_Parts:1711725
Changed lines of the file:
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@@
 <part name="H5" library="holes" library_urn="urn:adsk.eagle:library:237" deviceset="MOUNT-PAD-ROUND" device="3.6" package3d_urn="urn:adsk.eagle:package:14284/1"/>
 <part name="H6" library="holes" library_urn="urn:adsk.eagle:library:237" deviceset="MOUNT-PAD-ROUND" device="3.6" package3d_urn="urn:adsk.eagle:package:14284/1"/>
+<part name="IC1" library="SamacSys_Parts" deviceset="1711725" device=""/>
 </parts>
 <sheets>
@@
 <attribute name="VALUE" x="-83.566" y="254.0762" size="1.778" layer="96"/>
 </instance>
+<instance part="IC1" gate="G$1" x="-137.16" y="208.28" smashed="yes">
+<attribute name="NAME" x="-120.65" y="215.9" size="1.778" layer="95" align="center-left"/>
+<attribute name="VALUE" x="-120.65" y="213.36" size="1.778" layer="96" align="center-left"/>
+</instance>
 </instances>

Commit message: Platinenentwurf
Parts:
- removed H1, H2, H3, H4, H5, H6: MOUNT-PAD-ROUND3.6, holes:MOUNT-PAD-ROUND3.6
- removed Q1: SMMBT3904WT1G, SamacSys_Parts:SMMBT3904WT1G
- removed R16: 100K, adafruit:R-US_R1206
- removed R17: 7.5K, adafruit:R-US_R1206
- removed R5: (no value), adafruit:R-US_R1206
- removed SENSORIK: M20-9980545, SamacSys_Parts:M20-9980545
Connections:
- removed net CD_EN: CD74HCT.!1OE, CD74HCT.!2OE, CD74HCT.!4OE
- removed net CD_VCC: CD74HCT.VCC
- removed net INH_EXT: U2A.PA6
- removed net N$15: SENSORIK.6
- removed net N$21: J1.9
- removed net N$22: J1.10
- removed net N$23: J1.11
- removed net OUT_PA4: R3.1, SENSORIK.7
- removed net OUT_PA5: R5.1, SENSORIK.3
- removed net OUT_PA6: SENSORIK.5
- removed net OUT_PB1: R7.1, SENSORIK.1
- removed net PA4: R3.2, R4.1, U2A.PA4
- removed net PA5: R5.2, R6.1, U2A.PA5
- removed net PA8: Q1.C, R16.2, U2A.PA8
- removed net PB1: R7.2, R8.1, U2A.PB1
- removed net SS_VN: Q1.B, R17.1, SENSORIK.2
- new net L_1: R3.1
- new net L_2: R2.1
- new net PA1: R3.2, R4.1, U2A.PA1
- new net PC2: R7.2, R8.1, U2A.PC2
- new net T_1: R6.1, U2A.PC3
- new net U_RX: U2A.PA3
- new net U_TX: U2A.PA2
- new net Z_1: R7.1
- net GND: now also CD74HCT.!1OE, CD74HCT.!2OE, CD74HCT.!4OE; no longer Q1.E, R17.2, SENSORIK.4
- net INH: now also U2A.PC4; no longer U2A.PC2
- net IN_1: no longer U2A.PB11
- net IN_2: no longer U2A.PA1
- net IN_M_1: now also U2A.PB11
- net IN_M_2: now also U2A.PB10
- net IS_1: now also U2A.PB0; no longer U2A.PC0
- net IS_2: now also U2A.PB1; no longer U2A.PC1
- net NRST: now also J1.10
- net TRACESWO: now also J1.9
- net V12: no longer J1.12, R2.1
- net V33: no longer R16.1, SENSORIK.9
- net V5: now also CD74HCT.VCC
- net V_MOT_MIN: now also IC1.1; no longer J1.13
- net V_MOT_PL: now also IC1.2; no longer J1.14
Other:
- moved on the sheet: CD74HCT, IC1, J1

Commit message: Inventarliste added
Parts:
- removed R18, R19: 1k, adafruit:R-US_R1206
- added C16, C17, C18, C19: 220nF, adafruit:C-USC1206
- added J2, J3: 282836-2, SamacSys_Parts:282836-2
- added J4: M20-9990246, SamacSys_Parts:M20-9990246
- added R16: 220, adafruit:R-US_R1206
- added R17: 0, adafruit:R-US_R1206
- added R5: 100, adafruit:R-US_R1206
- added R_RS: 10, adafruit:R-US_R1206
- C11: value 4.7nF -> 4.7uF
- CH1, CH3: value 0.47uF -> 100nF
Connections:
- removed net BOOT0: R19.2, U2A.BOOT0
- removed net BOOT1: R18.2, U2A.PB2/BOOT1
- new net CAN_RS: CAN_T.RS, R_RS.1
- new net Q_IN: CQ2.1, QUARTZ.2, R17.2
- new net Q_OUT: CQ1.1, QUARTZ.1, R16.2
- net CANH: now also R5.2
- net CANL: now also R5.1
- net GND: now also C18.1, C19.1, J1.11, J3.1, R_RS.2, U2A.BOOT0, U2A.PB2/BOOT1; no longer CAN_T.RS, R18.1, R19.1
- net INH: no longer U2A.PC4
- net INH_M: now also U2A.PC4
- net L_1: now also J1.13, J2.2
- net L_2: now also J1.14, J2.1
- net OSC_IN: now also R17.1; no longer CQ2.1, QUARTZ.2
- net OSC_OUT: now also R16.1; no longer CQ1.1, QUARTZ.1
- net U_RX: now also J4.1
- net U_TX: now also J4.2
- net V12: now also C16.2, C17.2
- net V33: now also J3.2; no longer CD74HCT.!3OE
- net V5: now also J1.12
- net V_MOT_MIN: now also C17.1, C19.2
- net V_MOT_PL: now also C16.1, C18.2
Other:
- moved on the sheet: CQ1, CQ2, C_CAN, QUARTZ

Commit message: Platinenzeug
Parts:
- added C20: 1 uF, adafruit:C-USC1206
- added R15, R18: (no value), adafruit:R-US_R1206
- renumbered QUARTZ to QUARZ
Connections:
- new net PC5: R15.2, R18.1, U2A.PC5
- net GND: now also C20.2, R18.2
- net L_1: no longer J2.2
- net L_2: no longer J2.1
- net T_1: now also J2.1
- net V12: now also R15.1
- net V33: now also C20.1
- net Z_1: now also J2.2
Other:
- moved on the sheet: C1, C13, C2, C3, C4, CD74HCT, IC1, VREG_33, VREG_5

Commit message: Platinenzeug
Parts:
- removed R16: 220, adafruit:R-US_R1206
- removed R17: 0, adafruit:R-US_R1206
- added C21: 1uF, adafruit:C-USC1206
- added R19: 0, resistor:R-US_R0805
- added R20: 220, resistor:R-US_R0805
- added U$1: (no value), Nordic_nRF:INDUCTOR_0805_N
- R14, R9: value 1k -> 0.5k
Connections:
- new net VDDA: C12.1, C20.1, U$1.1, U2B.VDDA
- net CANH: now also J1.13; no longer J1.8
- net CANL: now also J1.14; no longer J1.7
- net GND: now also C21.2, J1.3, J1.8; no longer J1.11, J1.6
- net L_1: now also J1.7; no longer J1.13
- net L_2: now also J1.6; no longer J1.14
- net NRST: now also J1.11; no longer J1.10
- net OSC_IN: now also R19.2; no longer R17.1
- net OSC_OUT: now also R20.2; no longer R16.1
- net Q_IN: now also R19.1; no longer R17.2
- net Q_OUT: now also R20.1; no longer R16.2
- net SWCLK: now also J1.1; no longer J1.3
- net SWDIO: now also J1.10; no longer J1.2
- net TRACESWO: now also J1.12; no longer J1.9
- net T_1: now also C21.1
- net V33: now also J1.2, U$1.2; no longer C12.1, C20.1, J1.1, U2B.VDDA
- net V5: now also J1.9; no longer J1.12
