File: Platinenentwurf/testboard/BoardGeroutet/Board.brd (EAGLE design)
At the start: 88.8 x 50 mm, 61 parts, among them IC1 1711725, J1 1-776267-1, J2 282836-2, J3 282836-2, J4 M20-9990246

Commit message: Platinenzeugs
Routing:
- net V12: track 89.0 -> 87.4 mm
Other:
- board text added: "TSE-BOARD"
Changed lines of the file:
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@@
 <setting verticaltext="up"/>
 </settings>
-<grid distance="0.5" unitdist="mm" unit="mm" style="lines" multiple="1" display="yes" altdistance="5" altunitdist="mil" altunit="mil"/>
+<grid distance="1" unitdist="mm" unit="mm" style="lines" multiple="1" display="yes" altdistance="5" altunitdist="mil" altunit="mil"/>
 <layers>
-<layer number="1" name="Top" color="4" fill="1" visible="yes" active="yes"/>
+<layer number="1" name="Top" color="4" fill="1" visible="no" active="yes"/>
 <layer number="2" name="Route2" color="16" fill="1" visible="no" active="no"/>
 <layer number="3" name="Route3" color="17" fill="1" visible="no" active="no"/>
@@
 <layer number="14" name="Route14" color="22" fill="1" visible="no" active="no"/>
 <layer number="15" name="Route15" color="23" fill="1" visible="no" active="no"/>
-<layer number="16" name="Bottom" color="1" fill="1" visible="yes" active="yes"/>
+<layer number="16" name="Bottom" color="1" fill="1" visible="no" active="yes"/>
 <layer number="17" name="Pads" color="2" fill="1" visible="yes" active="yes"/>
 <layer number="18" name="Vias" color="2" fill="1" visible="yes" active="yes"/>
@@
 <layer number="23" name="tOrigins" color="15" fill="1" visible="yes" active="yes"/>
 <layer number="24" name="bOrigins" color="15" fill="1" visible="yes" active="yes"/>
-<layer number="25" name="tNames" color="7" fill="1" visible="no" active="yes"/>
+<layer number="25" name="tNames" color="7" fill="1" visible="yes" active="yes"/>
 <layer number="26" name="bNames" color="7" fill="1" visible="no" active="yes"/>
 <layer number="27" name="tValues" color="7" fill="1" visible="no" active="yes"/>
@@
 <dimension x1="0" y1="50" x2="0" y2="0" x3="-30" y3="25" textsize="1.778" layer="51"/>
 <dimension x1="0" y1="0" x2="88.8" y2="0" x3="44.4" y3="-30" textsize="1.778" layer="51"/>
+<text x="35" y="47" size="1" layer="21">TSE-BOARD</text>
 </plain>
 <attributes>
@@
 <attribute name="MOUSER_PART_NUMBER" value="815-ABLS-8.0MK4-T" x="-33.34" y="88.09" size="1.778" layer="27" rot="R180" display="off"/>
 <attribute name="MPN" value="ABLS-8.000MHZ-K4T" x="-33.34" y="88.09" size="1.778" layer="27" rot="R180" display="off"/>
-<attribute name="NAME" x="16.41433125" y="6.081" size="0.7" layer="25" rot="R180" align="center"/>
+<attribute name="NAME" x="19.41433125" y="4.081" size="0.7" layer="25" rot="R180" align="center"/>
 <attribute name="OC_FARNELL" value="2467758" x="-33.34" y="88.09" size="1.778" layer="27" rot="R180" display="off"/>
 <attribute name="VALUE" x="19.91433125" y="2.581" size="1.27" layer="27" rot="R180" align="center"/>
@@
 </element>
 <element name="C17" library="adafruit" library_urn="urn:adsk.eagle:library:420" package="C1206" package3d_urn="urn:adsk.eagle:package:6240335/1" value="220nF" x="60" y="23" smashed="yes">
-<attribute name="NAME" x="58.73" y="24.143" size="1.27" layer="25"/>
+<attribute name="NAME" x="57" y="22" size="0.7" layer="25" rot="R90"/>
 <attribute name="VALUE" x="58.73" y="20.587" size="1.27" layer="27"/>
 </element>
@@
 </element>
 <element name="R19" library="resistor" library_urn="urn:adsk.eagle:library:348" package="R0805" package3d_urn="urn:adsk.eagle:package:23553/2" value="0" x="15" y="9" smashed="yes" rot="R90">
-<attribute name="NAME" x="15.5" y="12.5" size="0.7" layer="25" rot="R180"/>
+<attribute name="NAME" x="16" y="13" size="0.7" layer="25" rot="R180"/>
 <attribute name="VALUE" x="17.54" y="8.365" size="1.27" layer="27" rot="R90"/>
 </element>
@@
 </element>
 <element name="R16" library="resistor" library_urn="urn:adsk.eagle:library:348" package="R0805" package3d_urn="urn:adsk.eagle:package:23553/2" value="220" x="53" y="24" smashed="yes" rot="R180">
-<attribute name="NAME" x="53.635" y="22.73" size="1.27" layer="25" rot="R180"/>
+<attribute name="NAME" x="54" y="26" size="0.7" layer="25" rot="R180"/>
 <attribute name="VALUE" x="53.635" y="26.54" size="1.27" layer="27" rot="R180"/>
 </element>
 <element name="R17" library="resistor" library_urn="urn:adsk.eagle:library:348" package="R0805" package3d_urn="urn:adsk.eagle:package:23553/2" value="220" x="46" y="15" smashed="yes" rot="R90">
-<attribute name="NAME" x="44.73" y="14.365" size="1.27" layer="25" rot="R90"/>
+<attribute name="NAME" x="45" y="18" size="0.7" layer="25"/>
 <attribute name="VALUE" x="48.54" y="14.365" size="1.27" layer="27" rot="R90"/>
 </element>
@@
 <vertex x="75" y="34.5"/>
 <vertex x="74.5" y="35"/>
-<vertex x="74.5" y="37.5"/>
-<vertex x="72" y="40"/>
-<vertex x="64.5" y="40"/>
-<vertex x="63.5" y="39"/>
+<vertex x="74.5" y="35.5"/>
+<vertex x="71" y="39"/>
+<vertex x="64.5" y="39"/>
+<vertex x="63.5" y="38"/>
 <vertex x="63.5" y="35.5"/>
-<vertex x="69.5" y="35.5"/>
-<vertex x="70.5" y="34.5"/>
-<vertex x="70.5" y="25"/>
-<vertex x="69.5" y="24"/>
-<vertex x="64.5" y="24"/>
-<vertex x="63.5" y="23"/>
+<vertex x="70" y="35.5"/>
+<vertex x="71.5" y="34"/>
+<vertex x="71.5" y="24"/>
+<vertex x="70" y="22.5"/>
+<vertex x="64.5" y="22.5"/>
+<vertex x="63.5" y="21.5"/>
 </polygon>
 <contactref element="J1" pad="4"/>
@@
 <wire x1="41" y1="39.5" x2="42.75" y2="41.25" width="0.5" layer="1"/>
 <wire x1="59" y1="43.6" x2="59" y2="38.26" width="0.5" layer="1"/>
-<wire x1="61.4" y1="23" x2="66.5" y2="23" width="0.5" layer="1"/>
-<wire x1="66.5" y1="23" x2="67" y2="22.5" width="0.5" layer="1"/>
+<wire x1="61.4" y1="23" x2="63.5" y2="23" width="0.5" layer="1"/>
+<wire x1="63.5" y1="23" x2="65" y2="21.5" width="0.5" layer="1"/>
 <wire x1="70.6" y1="17" x2="70.6" y2="20.4" width="0.5" layer="1"/>
 <wire x1="70.6" y1="20.4" x2="70.5" y2="20.5" width="0.5" layer="1"/>
@@
 <wire x1="20" y1="2" x2="41.5" y2="2" width="0.2" layer="16"/>
 <wire x1="41.5" y1="2" x2="42.384" y2="1.116" width="0.2" layer="16"/>
-<wire x1="67.616" y1="1.116" x2="67.75" y2="1.25" width="0.2" layer="16"/>
 <via x="69" y="2.5" extent="1-16" drill="0.508"/>
-<wire x1="67.75" y1="1.25" x2="69" y2="2.5" width="0.2" layer="16"/>
+<wire x1="67.616" y1="1.116" x2="69" y2="2.5" width="0.2" layer="16"/>
 <wire x1="69" y1="2.5" x2="70" y2="3.5" width="0.2" layer="1"/>
 <wire x1="70" y1="3.5" x2="70" y2="5" width="0.2" layer="1"/>
 <wire x1="4" y1="9" x2="2.5" y2="7.5" width="0.2" layer="1"/>
 <wire x1="2.884" y1="1.116" x2="19.116" y2="1.116" width="0.2" layer="1"/>
-<wire x1="42.384" y1="1.116" x2="67.616" y2="1.116" width="0.2" layer="16"/>
-<wire x1="75.530125" y1="1.21" x2="81.169875" y2="1.21" width="0.2" layer="16"/>
+<wire x1="42.384" y1="1.116" x2="67" y2="1.116" width="0.2" layer="16"/>
+<wire x1="67" y1="1.116" x2="67.616" y2="1.116" width="0.2" layer="16"/>
 <wire x1="86.76378125" y1="26.6025" x2="83.93621875" y2="26.6025" width="0.2" layer="16"/>
 <wire x1="83.93621875" y1="26.6025" x2="83.4975" y2="26.16378125" width="0.2" layer="16"/>
 <wire x1="83.4975" y1="26.16378125" x2="83.4975" y2="22.54904375" width="0.2" layer="16"/>
-<wire x1="67.75" y1="1.25" x2="75.490125" y2="1.25" width="0.2" layer="16"/>
-<wire x1="75.490125" y1="1.25" x2="75.530125" y2="1.21" width="0.2" layer="16"/>
-<wire x1="81.169875" y1="1.21" x2="87.39" y2="7.430125" width="0.2" layer="16"/>
 <wire x1="87.39" y1="7.430125" x2="87.39" y2="25.97628125" width="0.2" layer="16"/>
 <wire x1="87.39" y1="25.97628125" x2="86.76378125" y2="26.6025" width="0.2" layer="16"/>
@@
 <wire x1="29" y1="25.5" x2="29" y2="24.5" width="0.3" layer="1"/>
 <wire x1="29" y1="24.5" x2="29.5" y2="24" width="0.3" layer="1"/>
+<wire x1="67.616" y1="1.116" x2="81.075875" y2="1.116" width="0.2" layer="16"/>
+<wire x1="81.075875" y1="1.116" x2="87.39" y2="7.430125" width="0.2" layer="16"/>
 </signal>
 <signal name="V5">
@@
 <vertex x="59" y="37"/>
 <vertex x="51" y="37"/>
-<vertex x="51" y="32"/>
-<vertex x="41" y="32"/>
-<vertex x="40" y="31"/>
-<vertex x="40" y="27"/>
-<vertex x="41" y="26"/>
-<vertex x="48" y="26"/>
-<vertex x="49" y="27"/>
+<vertex x="51" y="30"/>
+<vertex x="42" y="30"/>
+<vertex x="41.5" y="29.5"/>
+<vertex x="41.5" y="27.5"/>
+<vertex x="42" y="27"/>
 <vertex x="59" y="27"/>
 </polygon>
@@
 <vertex x="59" y="37"/>
 <vertex x="51" y="37"/>
-<vertex x="51" y="32"/>
-<vertex x="41" y="32"/>
-<vertex x="40" y="31"/>
-<vertex x="40" y="27"/>
-<vertex x="41" y="26"/>
-<vertex x="48" y="26"/>
-<vertex x="49" y="27"/>
+<vertex x="51" y="27"/>
 <vertex x="59" y="27"/>
 </polygon>
@@
 <contactref element="C19" pad="2"/>
 <polygon width="0.1524" layer="1" thermals="no">
-<vertex x="41" y="25"/>
-<vertex x="48" y="25"/>
-<vertex x="49" y="24"/>
-<vertex x="49" y="22"/>
+<vertex x="42" y="24"/>
+<vertex x="47" y="24"/>
 <vertex x="50" y="21"/>
 <vertex x="59" y="21"/>
 <vertex x="59" y="11"/>
-<vertex x="52" y="11"/>
 <vertex x="51" y="11"/>
-<vertex x="51" y="16"/>
-<vertex x="49" y="16"/>
-<vertex x="45" y="20"/>
-<vertex x="42" y="20"/>
-<vertex x="41" y="20"/>
-<vertex x="40" y="21"/>
-<vertex x="40" y="24"/>
+<vertex x="51" y="18"/>
+<vertex x="49" y="18"/>
+<vertex x="46" y="21"/>
+<vertex x="42" y="21"/>
+<vertex x="41.5" y="21.5"/>
+<vertex x="41.5" y="23.5"/>
 </polygon>
 <wire x1="43" y1="23" x2="43" y2="17.4" width="0.5" layer="1"/>
@@
 <wire x1="57" y1="23" x2="56.5" y2="22.5" width="0.5" layer="1"/>
 <polygon width="0.2" layer="16" thermals="no">
-<vertex x="41" y="25"/>
-<vertex x="48" y="25"/>
-<vertex x="49" y="24"/>
-<vertex x="49" y="22"/>
-<vertex x="50" y="21"/>
+<vertex x="51" y="21"/>
 <vertex x="59" y="21"/>
 <vertex x="59" y="11"/>
 <vertex x="51.3" y="11"/>
 <vertex x="51" y="11.3"/>
-<vertex x="51" y="16"/>
-<vertex x="49" y="16"/>
-<vertex x="45" y="20"/>
-<vertex x="41" y="20"/>
-<vertex x="40" y="21"/>
-<vertex x="40" y="24"/>
 </polygon>
 <wire x1="56.5" y1="22.5" x2="56.5" y2="19" width="0.5" layer="1"/>

Commit message: Platinenzeugs
Parts:
- CQ1, CQ2: value 22pF -> 18pF
Changed lines of the file:
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@@
 <grid distance="1" unitdist="mm" unit="mm" style="lines" multiple="1" display="yes" altdistance="5" altunitdist="mil" altunit="mil"/>
 <layers>
-<layer number="1" name="Top" color="4" fill="1" visible="no" active="yes"/>
+<layer number="1" name="Top" color="4" fill="1" visible="yes" active="yes"/>
 <layer number="2" name="Route2" color="16" fill="1" visible="no" active="no"/>
 <layer number="3" name="Route3" color="17" fill="1" visible="no" active="no"/>
@@
 <layer number="20" name="Dimension" color="24" fill="1" visible="yes" active="yes"/>
 <layer number="21" name="tPlace" color="7" fill="1" visible="yes" active="yes"/>
-<layer number="22" name="bPlace" color="7" fill="1" visible="no" active="yes"/>
+<layer number="22" name="bPlace" color="7" fill="1" visible="yes" active="yes"/>
 <layer number="23" name="tOrigins" color="15" fill="1" visible="yes" active="yes"/>
 <layer number="24" name="bOrigins" color="15" fill="1" visible="yes" active="yes"/>
@@
 <dimension x1="0" y1="50" x2="0" y2="0" x3="-30" y3="25" textsize="1.778" layer="51"/>
 <dimension x1="0" y1="0" x2="88.8" y2="0" x3="44.4" y3="-30" textsize="1.778" layer="51"/>
-<text x="35" y="47" size="1" layer="21">TSE-BOARD</text>
+<text x="86" y="39" size="1" layer="21" rot="R90">TSE-BOARD</text>
 </plain>
 <attributes>
@@
 <attribute name="VALUE" x="70.73" y="14.587" size="1.27" layer="27"/>
 </element>
-<element name="CQ1" library="adafruit" library_urn="urn:adsk.eagle:library:420" package="C0805" package3d_urn="urn:adsk.eagle:package:6240337/1" value="22pF" x="21" y="9" smashed="yes" rot="R90">
+<element name="CQ1" library="adafruit" library_urn="urn:adsk.eagle:library:420" package="C0805" package3d_urn="urn:adsk.eagle:package:6240337/1" value="18pF" x="21" y="9" smashed="yes" rot="R90">
 <attribute name="NAME" x="20" y="6" size="0.7" layer="25"/>
 <attribute name="VALUE" x="23.286" y="8.111" size="1.27" layer="27" rot="R90"/>
 </element>
-<element name="CQ2" library="adafruit" library_urn="urn:adsk.eagle:library:420" package="C0805" package3d_urn="urn:adsk.eagle:package:6240337/1" value="22pF" x="12" y="9" smashed="yes" rot="R90">
+<element name="CQ2" library="adafruit" library_urn="urn:adsk.eagle:library:420" package="C0805" package3d_urn="urn:adsk.eagle:package:6240337/1" value="18pF" x="12" y="9" smashed="yes" rot="R90">
 <attribute name="NAME" x="13" y="13" size="0.7" layer="25" rot="R180"/>
 <attribute name="VALUE" x="14.286" y="8.111" size="1.27" layer="27" rot="R90"/>

Commit message: Platinenzeugs
Routing:
- net SR2: track 29.8 -> 30.4 mm
- net GND: vias 22 -> 34
Changed lines of the file:
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@@
 <setting verticaltext="up"/>
 </settings>
-<grid distance="1" unitdist="mm" unit="mm" style="lines" multiple="1" display="yes" altdistance="5" altunitdist="mil" altunit="mil"/>
+<grid distance="0.5" unitdist="mm" unit="mm" style="lines" multiple="1" display="yes" altdistance="5" altunitdist="mil" altunit="mil"/>
 <layers>
 <layer number="1" name="Top" color="4" fill="1" visible="yes" active="yes"/>
@@
 <layer number="14" name="Route14" color="22" fill="1" visible="no" active="no"/>
 <layer number="15" name="Route15" color="23" fill="1" visible="no" active="no"/>
-<layer number="16" name="Bottom" color="1" fill="1" visible="no" active="yes"/>
+<layer number="16" name="Bottom" color="1" fill="1" visible="yes" active="yes"/>
 <layer number="17" name="Pads" color="2" fill="1" visible="yes" active="yes"/>
 <layer number="18" name="Vias" color="2" fill="1" visible="yes" active="yes"/>
@@
 <via x="15.405" y="17.745" extent="1-16" drill="0.508"/>
 <via x="22.035" y="11.115" extent="1-16" drill="0.508"/>
-<polygon width="0.1524" layer="1" rank="2">
+<polygon width="0.1524" layer="1" thermals="no" rank="2">
 <vertex x="-1" y="51"/>
 <vertex x="-1" y="-1"/>
@@
 <vertex x="90" y="51"/>
 </polygon>
-<polygon width="0.1524" layer="16" rank="2">
+<polygon width="0.1524" layer="16" thermals="no" rank="2">
 <vertex x="-1" y="51"/>
 <vertex x="-1" y="-1"/>
@@
 <via x="35.5" y="17" extent="1-16" drill="0.508"/>
 <via x="38.5" y="22" extent="1-16" drill="0.508"/>
+<via x="67" y="24" extent="1-16" drill="0.508"/>
+<via x="69" y="24" extent="1-16" drill="0.508"/>
+<via x="70" y="25" extent="1-16" drill="0.508"/>
+<via x="64" y="27" extent="1-16" drill="0.508"/>
+<via x="66" y="27" extent="1-16" drill="0.508"/>
+<via x="62" y="14" extent="1-16" drill="0.508"/>
+<via x="62" y="16" extent="1-16" drill="0.508"/>
+<via x="65.5" y="11" extent="1-16" drill="0.508"/>
+<via x="63.5" y="11" extent="1-16" drill="0.508"/>
+<via x="65" y="23.5" extent="1-16" drill="0.508"/>
+<via x="70.5" y="26.5" extent="1-16" drill="0.508"/>
+<via x="60.5" y="9.5" extent="1-16" drill="0.508"/>
 </signal>
 <signal name="CAN1_RX">
@@
 <polygon width="0.2" layer="16" thermals="no">
 <vertex x="59" y="37"/>
-<vertex x="51" y="37"/>
-<vertex x="51" y="27"/>
+<vertex x="41" y="37"/>
+<vertex x="41" y="27"/>
 <vertex x="59" y="27"/>
 </polygon>
@@
 <wire x1="58.6" y1="23" x2="57" y2="23" width="0.5" layer="1"/>
 <wire x1="57" y1="23" x2="56.5" y2="22.5" width="0.5" layer="1"/>
-<polygon width="0.2" layer="16" thermals="no">
-<vertex x="51" y="21"/>
-<vertex x="59" y="21"/>
-<vertex x="59" y="11"/>
-<vertex x="51.3" y="11"/>
-<vertex x="51" y="11.3"/>
-</polygon>
 <wire x1="56.5" y1="22.5" x2="56.5" y2="19" width="0.5" layer="1"/>
 <via x="52" y="19.5" extent="1-16" drill="0.508"/>
@@
 <via x="53.5" y="13.5" extent="1-16" drill="0.508"/>
 <via x="53.5" y="12" extent="1-16" drill="0.508"/>
+<polygon width="0.1524" layer="16" thermals="no">
+<vertex x="59" y="21"/>
+<vertex x="50.5" y="21"/>
+<vertex x="50" y="21"/>
+<vertex x="47" y="24"/>
+<vertex x="42" y="24"/>
+<vertex x="41.5" y="23.5"/>
+<vertex x="41.5" y="21.5"/>
+<vertex x="41.5" y="18.5"/>
+<vertex x="44.5" y="15.5"/>
+<vertex x="44.5" y="14"/>
+<vertex x="45" y="13.5"/>
+<vertex x="45.5" y="13.5"/>
+<vertex x="46.5" y="12.5"/>
+<vertex x="49.5" y="12.5"/>
+<vertex x="50" y="12.5"/>
+<vertex x="51.5" y="11"/>
+<vertex x="59" y="11"/>
+</polygon>
 </signal>
 <signal name="IN_M_1">
@@
 <contactref element="HB_2" pad="5"/>
 <contactref element="R17" pad="2"/>
-<wire x1="60.5" y1="15.5" x2="60.5" y2="11" width="0.2" layer="1"/>
+<wire x1="60.5" y1="16.5" x2="60.5" y2="11" width="0.2" layer="1"/>
 <wire x1="60.5" y1="11" x2="58.5" y2="9" width="0.2" layer="1"/>
 <wire x1="51.65463125" y1="9" x2="49.76463125" y2="10.89" width="0.2" layer="1"/>
@@
 <wire x1="49.11" y1="10.89" x2="48" y2="12" width="0.2" layer="1"/>
 <wire x1="48" y1="12" x2="48" y2="15" width="0.2" layer="1"/>
-<wire x1="65.1" y1="17.27" x2="62.27" y2="17.27" width="0.2" layer="1"/>
-<wire x1="62.27" y1="17.27" x2="60.5" y2="15.5" width="0.2" layer="1"/>
+<wire x1="65.1" y1="17.27" x2="61.27" y2="17.27" width="0.2" layer="1"/>
+<wire x1="61.27" y1="17.27" x2="60.5" y2="16.5" width="0.2" layer="1"/>
+</signal>
+<signal name="N$1">
+<via x="68" y="32" extent="1-16" drill="0.508"/>
+</signal>
+<signal name="N$2">
+<via x="70" y="32" extent="1-16" drill="0.508"/>
 </signal>
 </signals>
