File: Platinenentwurf/testboard/BoardGeroutet/Board.sch (EAGLE design)
At the start: 61 parts, among them IC1 1711725, J1 1-776267-1, J2 282836-2, J3 282836-2, J4 M20-9990246

Commit message: Platinenzeugs
Parts:
- CQ1, CQ2: value 22pF -> 18pF
Changed lines of the file:
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@@
 <part name="C12" library="adafruit" library_urn="urn:adsk.eagle:library:420" deviceset="C-US" device="C1206" package3d_urn="urn:adsk.eagle:package:6240335/1" value="100nF"/>
 <part name="C11" library="adafruit" library_urn="urn:adsk.eagle:library:420" deviceset="C-US" device="C1206" package3d_urn="urn:adsk.eagle:package:6240335/1" value="4.7uF"/>
-<part name="CQ1" library="adafruit" library_urn="urn:adsk.eagle:library:420" deviceset="C-US" device="C0805" package3d_urn="urn:adsk.eagle:package:6240337/1" value="22pF"/>
-<part name="CQ2" library="adafruit" library_urn="urn:adsk.eagle:library:420" deviceset="C-US" device="C0805" package3d_urn="urn:adsk.eagle:package:6240337/1" value="22pF"/>
+<part name="CQ1" library="adafruit" library_urn="urn:adsk.eagle:library:420" deviceset="C-US" device="C0805" package3d_urn="urn:adsk.eagle:package:6240337/1" value="18pF"/>
+<part name="CQ2" library="adafruit" library_urn="urn:adsk.eagle:library:420" deviceset="C-US" device="C0805" package3d_urn="urn:adsk.eagle:package:6240337/1" value="18pF"/>
 <part name="C_CAN" library="adafruit" library_urn="urn:adsk.eagle:library:420" deviceset="C-US" device="C1206" package3d_urn="urn:adsk.eagle:package:6240335/1" value="100nF"/>
 <part name="C1" library="adafruit" library_urn="urn:adsk.eagle:library:420" deviceset="C-US" device="C1206" package3d_urn="urn:adsk.eagle:package:6240335/1" value="4.7uF"/>
@@
 </instance>
 <instance part="C15" gate="G$1" x="-58.42" y="111.76" smashed="yes">
-<attribute name="NAME" x="-61.595" y="105.156" size="1.778" layer="95" rot="R90"/>
-<attribute name="VALUE" x="-61.849" y="112.776" size="1.778" layer="96" rot="R90"/>
+<attribute name="NAME" x="-59.055" y="105.156" size="1.778" layer="95" rot="R90"/>
+<attribute name="VALUE" x="-59.309" y="112.776" size="1.778" layer="96" rot="R90"/>
 </instance>
 <instance part="J1" gate="G$1" x="76.2" y="180.34" smashed="yes" rot="R270">
@@
 <instance part="R17" gate="G$1" x="-66.04" y="109.22" smashed="yes" rot="R90">
 <attribute name="NAME" x="-67.5386" y="105.41" size="1.778" layer="95" rot="R90"/>
-<attribute name="VALUE" x="-62.738" y="105.41" size="1.778" layer="96" rot="R90"/>
+<attribute name="VALUE" x="-70.358" y="105.41" size="1.778" layer="96" rot="R90"/>
 </instance>
 </instances>

Commit message: Board
Parts:
- C21: value 1uF -> 220nF
Changed lines of the file:
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@@
 <part name="R18" library="adafruit" library_urn="urn:adsk.eagle:library:420" deviceset="R-US_" device="R1206" package3d_urn="urn:adsk.eagle:package:6240569/1"/>
 <part name="GND23" library="supply1" library_urn="urn:adsk.eagle:library:371" deviceset="GND" device=""/>
-<part name="C21" library="adafruit" library_urn="urn:adsk.eagle:library:420" deviceset="C-US" device="C1206" package3d_urn="urn:adsk.eagle:package:6240335/1" value="1uF"/>
+<part name="C21" library="adafruit" library_urn="urn:adsk.eagle:library:420" deviceset="C-US" device="C1206" package3d_urn="urn:adsk.eagle:package:6240335/1" value="220nF"/>
 <part name="L1" library="Nordic_nRF" library_urn="urn:adsk.eagle:library:169009" deviceset="INDUCTOR" device="_0805_N" package3d_urn="urn:adsk.eagle:package:2593736/1"/>
 <part name="R19" library="resistor" library_urn="urn:adsk.eagle:library:348" deviceset="R-US_" device="R0805" package3d_urn="urn:adsk.eagle:package:23553/2" value="0"/>
